File: cad/board/board.kicad_sch (KiCad schematic)
At the start: 47 parts, among them IC1 MAX17048G+T10, J1 USB_C_Receptacle_USB2.0_16P, J2 LiPo (min 500mAh), J3 Conn_02x11_Odd_Even, Q1 DMP2045U, U1 ESP32-C6-MINI-1, U2 USBLC6-2SC6, U3 AP2112K-3.3, U4 MCP73831-2-OT

Commit message: Extend board to include new peripherals
Parts:
- removed J3: Conn_02x11_Odd_Even, Connector_PinHeader_2.54mm:PinHeader_2x11_P2.54mm_Vertical, symbol Connector_Generic:Conn_02x11_Odd_Even
- removed Q1: DMP2045U, Package_TO_SOT_SMD:TSOT-23, symbol Simulation_SPICE:PMOS
- added C10: 100nF, Capacitor_SMD:C_0603_1608Metric, symbol Device:C
- added C11, C12: 1uF, Capacitor_SMD:C_0603_1608Metric, symbol Device:C
- added Q1: DMP2045U, Package_TO_SOT_SMD:TSOT-23, symbol Transistor_FET:Q_PMOS_GSD
- added R13, R15: 100, Resistor_SMD:R_0603_1608Metric, symbol Device:R
- added R14, R16: 10K, Resistor_SMD:R_0603_1608Metric, symbol Device:R
- added S1, S2: PTS845VM20PSMTR4_LFS, Imports:PTS845VM20PSMTR4LFS, symbol PTS845VM20PSMTR4:PTS845VM20PSMTR4_LFS
- added VR1, VR2: PTV09A-4220U-B103, Imports:PTV09A4220FB103, symbol PTV09A-4220F-B103:PTV09A-4220F-B103
- R11, R12: Link https://www.digikey.de/de/products/detail/stackpole-electronics-inc/RMCF0603FT10K0/1761235 -> https://www.digikey.de/de/products/detail/stackpole-electronics-inc/RMCF0603FT4K70/1760998
Connections:
- net +3.3V: now also R14.1, R16.1
- net GND: now also C10.2, C11.2, C12.2, S1.2 (NO), S1.MP1, S1.MP2, S2.2 (NO), S2.MP1, S2.MP2, VR1.3 (CW), VR1.4 (MH1), VR1.5 (MH2), VR2.3 (CW), VR2.4 (MH1), VR2.5 (MH2)
- net IO0: now also VR1.2 (WIPER)
- net IO1: now also VR2.2 (WIPER)
- net IO2: now also R13.1, R14.2, S1.1 (COM_1), S1.3 (COM_2)
- net IO3: now also R15.1, R16.2, S2.1 (COM_1), S2.3 (COM_2)
- net VBAT: now also C10.1, Q1.3 (D)
- net VBUS: now also Q1.1 (G)
- net at C4.1, C6.1, D2.1 (K)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: now also Q1.2 (S)
- new net: C12.1, R15.2
- new net: C11.1, R13.2
- new net +3V3: VR1.1 (CCW), VR2.1 (CCW)
Other:
- note added: "Peripherals"
- note removed: "Connections"
- title: ESP32 C6 Prototype Board -> ESP32C6 Drawboard
